File: RF-Arduino-Pro-Mini.kicad_pcb (KiCad board)
At the start: 2 copper layers, 20.3 x 47 mm, 40 parts, among them Q1 8/16/20MHz, U1 ATmega328P-AU, U2 MIC5205-3.3YM5, X1 16 MHZ

Commit message: first update after v1 release
Parts:
- added REF**: PinHeader_1x01_P1.27mm_Vertical, Connector_PinHeader_1.27mm:PinHeader_1x01_P1.27mm_Vertical, F.Cu at (133.6, 85.6)
- added REF**: PinHeader_1x01_P1.27mm_Vertical, Connector_PinHeader_1.27mm:PinHeader_1x01_P1.27mm_Vertical, F.Cu at (129.8, 123.7)
- added REF**: PinHeader_1x01_P1.27mm_Vertical, Connector_PinHeader_1.27mm:PinHeader_1x01_P1.27mm_Vertical, F.Cu at (118.5, 128.6)
- _A1: footprint RF_Antenna:Texas_SWRA117D_2.4GHz_Right -> RF-Arduino-Pro-Mini:ANT-2.45-CHP
- moved _A1 5.32 mm to (123.2, 129.0), turned to 270 degrees
- moved _C2 3.20 mm to (118.1, 114.8), turned to 180 degrees
- moved _C5 1.68 mm to (124.8, 124.0)
- moved _C7 1.49 mm to (128.7, 118.5), turned to 0 degrees
- moved _C3 1.19 mm to (121.0, 122.4), turned to 180 degrees
- moved _C6 1.02 mm to (126.4, 124.4), turned to 0 degrees
- moved _R2 0.97 mm to (128.6, 121.5)
- moved _C8 0.90 mm to (128.1, 120.0)
- moved _C9 0.90 mm to (129.2, 120.0)
- moved _L2 0.89 mm to (123.2, 123.5), turned to 180 degrees
- moved _L3 0.82 mm to (125.8, 122.9)
- moved _U1 0.81 mm to (124.6, 119.3)
- moved _L1 0.81 mm to (124.3, 122.4)
- moved _R1 0.71 mm to (121.2, 120.0)
- moved _C4 0.69 mm to (121.0, 123.5), turned to 180 degrees
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Connections:
- _A1 pad 2: GND -> Net-(_A1-Pad2)
Routing:
- net GND: track 99.9 -> 102.8 mm, vias 22 -> 37
- net Net-(_A1-Pad1): track 1.83 -> 3.67 mm
- net D9: track 23.5 -> 25.1 mm
- net Net-(_C3-Pad1): track 3.61 -> 5.00 mm
- net MISO: track 21.5 -> 20.7 mm
- net SCK: track 17.8 -> 17.1 mm
- net /AREF: track 13.7 -> 13.1 mm
Other:
- board size 20.3 x 47 mm -> 21.6 x 48.3 mm
- board text added: "RF Pro Mini rev. 02.00"
