File: RF-Arduino-Pro-Mini.sch (KiCad schematic (older format))
At the start: 40 parts, among them Q1 8/16/20MHz, U1 ATmega328P-AU, U2 MIC5205-3.3YM5, X1 16 MHZ

Commit message: first update after v1 release
Parts:
- _A1: footprint RF_Antenna:Texas_SWRA117D_2.4GHz_Right -> RF-Arduino-Pro-Mini:ANT-2.45-CHP
Connections:
- net GND: no longer _A1.2 (Shield)
Changed lines of the file:
@@
 F 0 "_A1" V 12686 6530 50  0000 L CNN
 F 1 "Antenna" V 12800 6250 50  0000 L CNN
-F 2 "RF_Antenna:Texas_SWRA117D_2.4GHz_Right" H 12700 6400 50  0001 C CNN
+F 2 "RF-Arduino-Pro-Mini:ANT-2.45-CHP" H 12700 6400 50  0001 C CNN
 F 3 "~" H 12700 6400 50  0001 C CNN
 	1    12700 6300
 	0    1    1    0
 $EndComp
-$Comp
-L power:GND #PWR0132
-U 1 1 5E7E413C
-P 12500 6400
-F 0 "#PWR0132" H 12500 6150 50  0001 C CNN
-F 1 "GND" H 12505 6227 50  0000 C CNN
-F 2 "" H 12500 6400 50  0001 C CNN
-F 3 "" H 12500 6400 50  0001 C CNN
-	1    12500 6400
-	1    0    0    -1
-$EndComp
 Wire Wire Line
